File: hardware/motherboard.kicad_pcb (KiCad board)
At the start: 2 copper layers, 200 x 150 mm, 319 parts, among them J1 24 V DC input, J10 AX0: EN, STEP, DIR, GND, J11 AX1: EN, STEP, DIR, GND, J12 General outputs 0-7; pin9 fie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, J13 Encoder 0: +5,A,B,Z,GND, J14 Encoder 1: +5,A,B,Z,GND, J15 Encoder 2: +5,A,B,Z,GND, J16 Keyboard KIN0-7 / KOUT0-7, J17 Keyboard power/reference, J18 I2C0, J19 Full-size SD, SPI, J2 Backlight: +12V, GND, PWM, sw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, J20 ESP-01S socket, J22 LCD LVDS 2x10, 2.00 mm, J24 AI0/GND/AI1/GND/AI2/GND, J25 0-10 V outputs 0-3; pin 1 = c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, J26 Dedicated START button input, J27 Expansion inputs 4-7; 1=GND, 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, J28 AX2: EN, STEP, DIR, GND, J29 AX3: EN, STEP, DIR, GND, J30 AX4: EN, STEP, DIR, GND, J31 Motion AUX open-drain output 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, J32 General outputs 8-15; DO_COM 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, J33 General outputs field +V and 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, J34 PLC positions 5-8 of J7 bank;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, J35 PLC positions 5-8 of J8 bank;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, J36 MicroSD alternative, SPI, J4 SWD, J5 Dedicated E-stop loop, J6 Dedicated HOLD button input, J7 PLC inputs 1-8; alternating i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, J8 PLC inputs 9-16; alternating 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, J9 Expansion inputs 0-3; 1=GND, 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, Q5 BSS138, Q6 BSS138, Q7 BSS138, Q8 BSS138, SW2 ESP_PROG, U1 LMR36510ADDAR, U10 74HC595D, U11 74HC595D, U12 74HC595D, U13 74HC595D, U18 LTV-847S, U19 LTV-847S, U2 AMS1117-3.3, U20 LTV-847S, U21 LTV-847S, U24 SN74AHCT541DW, U25 SN74AHCT541DW, U26 ULN2003ADR, U27 ULN2003ADR, U28 SN74AHCT541DW, U3 LMR36510ADDAR, U34 AMS1117-3.3, U35 EL3H7, U36 EL3H7, U37 L78L12ACUTR, U38 TLV2374IDR, U39 EL3H7, U40 TBA2-0512, U41 DS90LV047A, U6 74HC165D, U7 74HC165D, U8 74HC165D, U9 74HC165D

Commit message: Add buck thermal vias and refresh 3D renders
Routing:
- net GND: vias 94 -> 106
Changed lines of the file:
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@@
+	)
+	(via
+		(at 186.75 129.6)
+		(size 0.6)
+		(drill 0.3)
+		(layers "F.Cu" "B.Cu")
+		(net "GND")
 	)
 	(via
@@
 	)
 	(via
+		(at 187.95 127.6)
+		(size 0.6)
+		(drill 0.3)
+		(layers "F.Cu" "B.Cu")
+		(net "GND")
+	)
+	(via
 		(at 193.175 78.925)
 		(size 0.6)
@@
 	)
 	(via
+		(at 187.7 107.675)
+		(size 0.6)
+		(drill 0.3)
+		(layers "F.Cu" "B.Cu")
+		(net "GND")
+	)
+	(via
 		(at 58.1 45.5)
 		(size 0.6)
@@
 	)
 	(via
+		(at 186.75 128.6)
+		(size 0.6)
+		(drill 0.3)
+		(layers "F.Cu" "B.Cu")
+		(net "GND")
+	)
+	(via
 		(at 61.8 28.2)
 		(size 0.6)
@@
 	)
 	(via
+		(at 187.7 108.675)
+		(size 0.6)
+		(drill 0.3)
+		(layers "F.Cu" "B.Cu")
+		(net "GND")
+	)
+	(via
 		(at 46.85 118.9)
 		(size 0.6)
@@
 	)
 	(via
+		(at 186.75 127.6)
+		(size 0.6)
+		(drill 0.3)
+		(layers "F.Cu" "B.Cu")
+		(net "GND")
+	)
+	(via
 		(at 46.9 75.55)
 		(size 0.6)
@@
 	)
 	(via
+		(at 186.5 108.675)
+		(size 0.6)
+		(drill 0.3)
+		(layers "F.Cu" "B.Cu")
+		(net "GND")
+	)
+	(via
 		(at 45.3 65.0625)
 		(size 0.6)
@@
 	)
 	(via
+		(at 187.95 129.6)
+		(size 0.6)
+		(drill 0.3)
+		(layers "F.Cu" "B.Cu")
+		(net "GND")
+	)
+	(via
 		(at 46.45 89.65)
 		(size 0.6)
@@
 	)
 	(via
+		(at 187.7 106.675)
+		(size 0.6)
+		(drill 0.3)
+		(layers "F.Cu" "B.Cu")
+		(net "GND")
+	)
+	(via
 		(at 115.282 45.513)
 		(size 0.6)
@@
 	)
 	(via
+		(at 186.5 107.675)
+		(size 0.6)
+		(drill 0.3)
+		(layers "F.Cu" "B.Cu")
+		(net "GND")
+	)
+	(via
+		(at 186.375 46.775)
+		(size 0.6)
+		(drill 0.3)
+		(layers "F.Cu" "B.Cu")
+		(net "GND")
+	)
+	(via
 		(at 186.45 51.65)
 		(size 0.6)
@@
 		(size 0.6)
 		(drill 0.3)
+		(layers "F.Cu" "B.Cu")
+		(net "GND")
+	)
+	(via
+		(at 187.95 128.6)
+		(size 0.6)
+		(drill 0.3)

Commit message: BOM simplification
Parts:
- added R128: 100k, R_1206_3216Metric, F.Cu at (192.8, 133.0)
- C105, C67: value 10uF -> 10uF 25V
- R127: value 9.09k -> 10k
- R70: value 34k -> 33k
- R71: value 46.4k -> 100k
- R72: value 20k -> 33k
- moved C88 32.7 mm to (157.2, 40.0), turned to 90 degrees
- moved C89 25.9 mm to (161.0, 45.1), turned to 0 degrees
- moved U34 20.2 mm to (163.5, 40.0), turned to 0 degrees
- moved C69 11.0 mm to (170.4, 39.0), turned to 90 degrees
- moved J20 5.47 mm to (177.6, 40.6)
- moved C70 5.39 mm to (176.2, 37.2)
- moved SW2 4.63 mm to (178.6, 33.0)
- moved RN36 4.63 mm to (181.4, 45.8)
- moved R126 1.58 mm to (195.4, 133.0), turned to 90 degrees
- moved D1 0.78 mm to (190.3, 137.7)
- moved R127 0.58 mm to (188.7, 132.4)
Routing:
- net +5V: track 445.0 -> 469.3 mm
- net +3V3: track 675.3 -> 668.2 mm
- net WIFI_TX: track 66.3 -> 71.8 mm
- net WIFI_RX: track 67.6 -> 73.1 mm
- net FB12: track 4.84 -> 8.35 mm
- net +12V_BL: track 66.8 -> 69.5 mm
- net +3V3_WIFI: track 33.0 -> 35.1 mm, vias 0 -> 1
- net WIFI_GPIO0: track 25.6 -> 24.3 mm
- net WIFI_GPIO2: track 4.42 -> 3.56 mm
- net WIFI_RST: track 7.22 -> 6.39 mm
- net WIFI_EN: track 4.35 -> 3.53 mm
- net VIN_FUSED: track 31.2 -> 31.8 mm, vias 3 -> 5
- net GND: vias 106 -> 99
