File: hardware/field_outputs.kicad_sch (KiCad schematic)
At the start: 46 parts, among them J10 AX0: EN, STEP, DIR, GND, J11 AX1: EN, STEP, DIR, GND, J12 General outputs 0-7; pin9 fie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, J28 AX2: EN, STEP, DIR, GND, J29 AX3: EN, STEP, DIR, GND, J30 AX4: EN, STEP, DIR, GND, J31 Motion AUX open-drain output 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, Q5 BSS138, U24 SN74AHCT541DW, U25 SN74AHCT541DW, U26 ULN2003ADR, U27 ULN2003ADR

Commit message: Update RP2350B PCB, pinout and fabrication rules
Parts:
- removed J12: General outputs 0-7; pin9 field +V, pin10 GND, Connector_Phoenix_MC:PhoenixContact_MCV_1,5_10-G-3.5_1x10_P3.50mm_Vertical, symbol Connector_Generic:Conn_01x10
- removed R112: 100R, Resistor_SMD:R_0805_2012Metric, symbol Device:R
- added D57: DO8, LED_SMD:LED_1206_3216Metric, symbol Device:LED
- added D58: DO9, LED_SMD:LED_1206_3216Metric, symbol Device:LED
- added D59: DO10, LED_SMD:LED_1206_3216Metric, symbol Device:LED
- added D60: DO11, LED_SMD:LED_1206_3216Metric, symbol Device:LED
- added D61: DO12, LED_SMD:LED_1206_3216Metric, symbol Device:LED
- added D62: DO13, LED_SMD:LED_1206_3216Metric, symbol Device:LED
- added D63: DO14, LED_SMD:LED_1206_3216Metric, symbol Device:LED
- added D64: DO15, LED_SMD:LED_1206_3216Metric, symbol Device:LED
- added J12: General outputs 0-7, Connector_Phoenix_MC:PhoenixContact_MCV_1,5_8-G-3.5_1x08_P3.50mm_Vertical, symbol Connector_Generic:Conn_01x08
- added J32: General outputs 8-15; DO_COM and GND are shared t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, Connector_Phoenix_MC:PhoenixContact_MCV_1,5_8-G-3.5_1x08_P3.50mm_Vertical, symbol Connector_Generic:Conn_01x08
- added J33: General outputs field +V and GND, Connector_Phoenix_MC:PhoenixContact_MCV_1,5_2-G-3.5_1x02_P3.50mm_Vertical, symbol Connector_Generic:Conn_01x02
- added Q6, Q7: BSS138, Package_TO_SOT_SMD:SOT-23, symbol Transistor_FET:Q_NMOS_GSD
- added R114, R116: 100R, Resistor_SMD:R_0805_2012Metric, symbol Device:R
- added R115, R117: 100k, Resistor_SMD:R_0805_2012Metric, symbol Device:R
- added R118, R119, R120, R121, R122, R123, R124, R125: 2.2k, Resistor_SMD:R_1206_3216Metric, symbol Device:R
- added RN30, RN31: 4x10k, Resistor_SMD:R_Array_Convex_4x0603, symbol LeanCam:ResistorPack04
- J31: value Motion AUX open-drain output and GND -> AUX open-drain output and GND
Connections:
- net AUX_GATE: now also RN16.6 (R3B)
- net BUFY0: now also RN8.6 (R3B); no longer RN8.1 (R1A)
- net BUFY1: now also RN8.5 (R4B); no longer RN8.2 (R2A)
- net BUFY12: now also RN11.5 (R4B); no longer RN11.1 (R1A)
- net BUFY13: now also RN11.6 (R3B); no longer RN11.2 (R2A)
- net BUFY14: now also RN11.7 (R2B); no longer RN11.3 (R3A)
- net BUFY15: now also RN11.8 (R1B); no longer RN11.4 (R4A)
- net BUFY2: now also RN8.8 (R1B); no longer RN8.3 (R3A)
- net BUFY3: now also RN8.7 (R2B); no longer RN8.4 (R4A)
- net BUFY4: now also RN9.2 (R2A); no longer RN9.1 (R1A)
- net BUFY5: now also RN9.1 (R1A); no longer RN9.2 (R2A)
- net BUFY6: now also RN9.4 (R4A); no longer RN9.3 (R3A)
- net BUFY7: now also RN9.3 (R3A); no longer RN9.4 (R4A)
- net BUFY8: now also RN10.2 (R2A); no longer RN10.1 (R1A)
- net BUFY9: now also RN10.1 (R1A); no longer RN10.2 (R2A)
- net DO0: now also U26.10 (O7), J12.1 (Pin_1); no longer U26.13 (O4)
- net DO1: now also U26.11 (O6), J12.2 (Pin_2); no longer U26.14 (O3)
- net DO2: now also U26.12 (O5), J12.3 (Pin_3); no longer U26.15 (O2)
- net DO3: now also U26.13 (O4), J12.4 (Pin_4); no longer U26.16 (O1)
- net DO4: now also U26.14 (O3), J12.5 (Pin_5); no longer U27.13 (O4)
- net DO5: now also U26.15 (O2), J12.6 (Pin_6); no longer U27.14 (O3)
- net DO6: now also U26.16 (O1), J12.7 (Pin_7); no longer U27.15 (O2)
- net DO7: now also U27.10 (O7), J12.8 (Pin_8); no longer U27.16 (O1)
- net DO_COM: now also J33.1 (Pin_1), R118.1, R119.1, R120.1, R121.1, R122.1, R123.1, R124.1, R125.1
- net GND: now also RN11.1 (R1A), RN11.2 (R2A), RN11.3 (R3A), RN11.4 (R4A), RN8.1 (R1A), RN8.2 (R2A), RN8.3 (R3A), RN8.4 (R4A), J33.2 (Pin_2), Q6.2 (S), Q7.2 (S), R115.2, R117.2, RN30.5 (R4B), RN30.6 (R3B), RN30.7 (R2B), RN30.8 (R1B), RN31.6 (R3B), RN31.7 (R2B), RN31.8 (R1B); no longer RN11.5 (R4B), RN11.6 (R3B), RN11.7 (R2B), RN11.8 (R1B), RN13.8 (R1B), RN8.5 (R4B), RN8.6 (R3B), RN8.7 (R2B), RN8.8 (R1B)
- net KOUT1: now also RN20.2 (R2A); no longer RN20.7 (R2B)
- net KOUT3: now also RN20.4 (R4A); no longer RN20.5 (R4B)
- net MOTION0: now also J10.1 (Pin_1); no longer J10.3 (Pin_3)
- net MOTION1: now also RN16.7 (R2B); no longer RN16.6 (R3B)
- net MOTION10: now also J29.2 (Pin_2), RN18.8 (R1B); no longer J29.1 (Pin_1), RN18.7 (R2B)
- net MOTION11: now also RN19.5 (R4B); no longer RN18.8 (R1B)
- net MOTION12: now also J30.1 (Pin_1), RN19.6 (R3B); no longer J30.3 (Pin_3), RN19.5 (R4B)
- net MOTION13: now also RN19.7 (R2B); no longer RN19.6 (R3B)
- net MOTION14: now also J30.3 (Pin_3), RN19.8 (R1B); no longer RN19.7 (R2B)
- net MOTION2: now also J10.3 (Pin_3), RN16.8 (R1B); no longer J11.2 (Pin_2), RN16.7 (R2B)
- net MOTION3: now also J11.1 (Pin_1), RN17.5 (R4B); no longer J10.1 (Pin_1), RN16.8 (R1B)
- net MOTION4: now also J11.2 (Pin_2), RN17.6 (R3B); no longer J11.1 (Pin_1), RN17.5 (R4B)
- net MOTION5: now also RN17.7 (R2B); no longer RN17.6 (R3B)
- net MOTION6: now also J28.1 (Pin_1), RN17.8 (R1B); no longer J28.3 (Pin_3), RN17.7 (R2B)
- net MOTION7: now also RN18.5 (R4B); no longer RN17.8 (R1B)
- net MOTION8: now also J28.3 (Pin_3), RN18.6 (R3B); no longer J29.2 (Pin_2), RN18.5 (R4B)
- net MOTION9: now also J29.1 (Pin_1), RN18.7 (R2B); no longer J28.1 (Pin_1), RN18.6 (R3B)
- net OUT16: now also RN12.4 (R4A), U26.7 (I7); no longer RN12.1 (R1A), U26.4 (I4)
- net OUT17: now also RN12.3 (R3A), U26.6 (I6); no longer RN12.2 (R2A), U26.3 (I3)
- net OUT18: now also RN12.2 (R2A), U26.5 (I5); no longer RN12.3 (R3A), U26.2 (I2)
- net OUT19: now also RN12.1 (R1A), U26.4 (I4); no longer RN12.4 (R4A), U26.1 (I1)
- net OUT20: now also RN13.4 (R4A), U26.3 (I3); no longer RN13.1 (R1A), U27.4 (I4)
- net OUT21: now also RN13.3 (R3A), U26.2 (I2); no longer RN13.2 (R2A), U27.3 (I3)
- net OUT22: now also RN13.2 (R2A), U26.1 (I1); no longer RN13.3 (R3A), U27.2 (I2)
- net OUT23: now also U27.7 (I7), RN30.4 (R4A); no longer RN13.4 (R4A), U27.1 (I1)
- net OUT24: now also U27.6 (I6), RN30.2 (R2A)
- net OUT25: now also RN20.7 (R2B), U27.5 (I5), RN30.3 (R3A); no longer RN20.2 (R2A)
- net OUT26: now also U27.4 (I4), RN30.1 (R1A)
- net OUT27: now also RN20.5 (R4B), U27.3 (I3), RN31.3 (R3A); no longer RN20.4 (R4A)
- net OUT28: now also U27.2 (I2), RN31.2 (R2A)
- net OUT29: now also U27.1 (I1), RN31.1 (R1A)
- net OUT30: now also R114.1
- net OUT31: now also R116.1
- net DO8: now reaches U27.11 (O6)
- net DO8: now also D57.1 (K), J32.1 (Pin_1)
- net DO9: now reaches U27.12 (O5)
- net DO9: now also D58.1 (K), J32.2 (Pin_2)
- removed net MOTION15: J30.1 (Pin_1), RN19.8 (R1B)
- new net DO10: D59.1 (K), J32.3 (Pin_3), U27.13 (O4)
- new net DO11: D60.1 (K), J32.4 (Pin_4), U27.14 (O3)
- new net DO12: D61.1 (K), J32.5 (Pin_5), U27.15 (O2)
- new net DO13: D62.1 (K), J32.6 (Pin_6), U27.16 (O1)
- new net DO14: D63.1 (K), J32.7 (Pin_7), Q6.3 (D)
- new net DO14_GATE: Q6.1 (G), R114.2, R115.1
- new net DO15: D64.1 (K), J32.8 (Pin_8), Q7.3 (D)
- new net DO15_GATE: Q7.1 (G), R116.2, R117.1
- new net DO_LED10_A: D59.2 (A), R120.2
- new net DO_LED11_A: D60.2 (A), R121.2
- new net DO_LED12_A: D61.2 (A), R122.2
- new net DO_LED13_A: D62.2 (A), R123.2
- new net DO_LED14_A: D63.2 (A), R124.2
- new net DO_LED15_A: D64.2 (A), R125.2
- new net DO_LED8_A: D57.2 (A), R118.2
- new net DO_LED9_A: D58.2 (A), R119.2
- no-connect marks 12 -> 4
