File: hardware/power.kicad_sch (KiCad schematic)
At the start: 38 parts, among them J1 24 V DC input, Q1 DMP1045U-7, U1 LMR36510ADDAR, U2 AMS1117-3.3

Commit message: Update RP2350B PCB, pinout and fabrication rules
Parts:
- removed C14, C16, C8: 10uF, Capacitor_SMD:C_1206_3216Metric, symbol Device:C
- removed C17, C77: 100nF, Capacitor_SMD:C_0805_2012Metric, symbol Device:C
- removed Q1: DMP1045U-7, Package_TO_SOT_SMD:SOT-23, symbol Transistor_FET:Q_PMOS_GSD
- added Q1: IRF7240PBF, Package_SO:SOIC-8_3.9x4.9mm_P1.27mm, symbol LeanCam:PMOS_SO8
Connections:
- net Q1_GATE: now also Q1.4 (G)
- net VIN_FUSED: now also Q1.5 (D1), Q1.6 (D2), Q1.7 (D3), Q1.8 (D4)
- net VIN_PROT: now also Q1.1 (S1), Q1.2 (S2), Q1.3 (S3)

Commit message: Update RP2350 board power and I/O design
Parts:
- removed C1: 10uF 50V, Capacitor_SMD:C_1206_3216Metric, symbol Device:C
- removed D2: MMSZ5242B, Diode_SMD:D_SOD-323, symbol Device:D_Zener
- removed Q1: IRF7240PBF, Package_SO:SOIC-8_3.9x4.9mm_P1.27mm, symbol LeanCam:PMOS_SO8
- removed R1: 100k, Resistor_SMD:R_1206_3216Metric, symbol Device:R
- added C107: 22uF 50V, Capacitor_SMD:C_1210_3225Metric, symbol Device:C
- added C108: 100nF 100V, Capacitor_SMD:C_1206_3216Metric, symbol Device:C
- added C109, C110, C111: 22uF 25V, Capacitor_SMD:C_1210_3225Metric, symbol Device:C
- added C112, C113: 100nF, Capacitor_SMD:C_0805_2012Metric, symbol Device:C
- added C114: 1uF, Capacitor_SMD:C_0805_2012Metric, symbol Device:C
- added D2, D3: SS16, Diode_SMD:D_SMA, symbol Device:D
- added J2: Backlight: +12V, GND, PWM, switched low-side, Connector_Phoenix_MC:PhoenixContact_MCV_1,5_4-G-3.5_1x04_P3.50mm_Vertical, symbol Connector_Generic:Conn_01x04
- added L2: 47uH 1.5A, Inductor_SMD:L_Bourns_SRN6045TA, symbol Device:L
- added Q8: BSS138, Package_TO_SOT_SMD:SOT-23, symbol Transistor_FET:Q_NMOS_GSD
- added R126: 100k, Resistor_SMD:R_1206_3216Metric, symbol Device:R
- added R127: 9.09k, Resistor_SMD:R_1206_3216Metric, symbol Device:R
- added R129, R131: 100R, Resistor_SMD:R_0805_2012Metric, symbol Device:R
- added R130: 100k, Resistor_SMD:R_0805_2012Metric, symbol Device:R
- added U3: LMR36510ADDAR, Package_SO:SOIC-8-1EP_3.9x4.9mm_P1.27mm_EP2.41x3.3mm, symbol Regulator_Switching:LMR36510ADDA
- C10: value 10uF -> 22uF 25V; footprint Capacitor_SMD:C_1206_3216Metric -> Capacitor_SMD:C_1210_3225Metric; MPN CL31 series 1206 X7R 10uF -> CL32 series 1210 X7R 22uF 25V
- C11, C6: value 22uF 10V -> 22uF 25V; MPN CL32 series 1210 X7R 22uF 10V -> CL32 series 1210 X7R 22uF 25V
- C3: value 10uF 50V -> 22uF 50V; footprint Capacitor_SMD:C_1206_3216Metric -> Capacitor_SMD:C_1210_3225Metric; MPN CL31 series 1206 X7R 10uF 50V -> CL32 series 1210 X7R 22uF 50V
- C90: value 22uF -> 22uF 25V; MPN CL32 series 1210 X7R 22uF -> CL32 series 1210 X7R 22uF 25V
Connections:
- net GND: now also C107.2, C108.2, C109.2, C110.2, C111.2, C112.2, C114.2, J2.2 (Pin_2), Q8.2 (S), R127.2, R130.2, U3.1 (PGND), U3.9 (PAD)
- net VIN_FUSED: now also D2.2 (A), D3.2 (A)
- net VIN_PROT: now also D2.1 (K)
- new net +12V_BL: C109.1, C110.1, C111.1, C112.1, J2.1 (Pin_1), L2.2, R126.1
- new net BL_LED_N: J2.4 (Pin_4), Q8.3 (D)
- new net BL_PWM: J2.3 (Pin_3), R131.2
- new net BL_PWM_MCU: R129.1, R131.1
- new net BL_SW_GATE: Q8.1 (G), R129.2, R130.1
- new net BUCK12_BST: C113.1, U3.7 (BOOT)
- new net BUCK12_SW: C113.2, L2.1, U3.8 (SW)
- new net FB12: R126.2, R127.1, U3.5 (FB)
- new net VCC12: C114.1, U3.6 (VCC)
- new net VIN_BL_PROT: C107.1, C108.1, D3.1 (K), U3.2 (VIN), U3.3 (EN)
- no-connect marks 0 -> 1

Commit message: Standardize passives and add microSD alternate
Parts:
- C10, C109, C11, C110, C111, C6, C90: value 22uF 25V -> 22uF 50V; MPN CL32 series 1210 X7R 22uF 25V -> CL32 series 1210 X7R 22uF 50V

Commit message: BOM simplification
Parts:
- added R128: 100k, Resistor_SMD:R_1206_3216Metric, symbol Device:R
- R127: value 9.09k -> 10k; MPN RC1206FR-07 1% 9.09k -> RC1206FR-07 1% 10k
- R70: value 34k -> 33k; MPN RC1206FR-07 1% 34k -> RC1206FR-07 1% 33k
- R71: value 46.4k -> 100k; MPN RC1206FR-07 1% 46.4k -> RC1206FR-07 1% 100k
- R72: value 20k -> 33k; MPN RC1206FR-07 1% 20k -> RC1206FR-07 1% 33k
Connections:
- net FB12: now also R128.1
- net GND: now also R128.2
